File: ActiveSpeakers_KiCad.kicad_pcb (KiCad board)
At the start: 2 copper layers, 232.1 x 150 mm, 281 parts, among them J1 ST-04M-160, J10 Conn_01x04, J11 Conn_02x05, J12 Conn_02x04, J13 Conn_01x04, J14 Conn_01x04, J15 Conn_01x04, J16 Conn_01x04, J17 Conn_01x04, J18 Conn_01x04, J19 Conn_01x04, J2 main.pwrin, J20 Conn_01x04, J21 Conn_01x04, J22 Conn_01x04, J23 Conn_01x04, J24 Conn_01x04, J25 Conn_01x04, J26 ISP, J27 Conn_01x04, J28 Conn_01x04, J29 Conn_01x04, J3 USB_B, J30 Conn_01x04, J31 Screw_Terminal_01x02, J32 Screw_Terminal_01x02, J4 Conn_02x05, J5 Conn_01x06, J6 Conn_01x04, J7 Conn_01x04, J8 Conn_01x06, J9 Conn_01x04, Q1 BC847, Q2 BC847, Q3 IRLML5203, Q4 IRLML5203, Q5 2N7002, Q6 BC857, U1 PCM2704, U10 TDA7419, U11 ATmega88PA-AU, U12 74HC595, U13 74HC595, U14 74HC595, U15 TDA7498, U2 FE1.1S, U3 CH340G, U4 78S05, U5 L7812, U6 L78L33_SOT89, U7 L7809, U8 LM75B, U9 TDA7317, Y1 12MHz, Y2 12MHz, Y3 12MHz, Y4 16MHz

Commit message: upd
Connections:
- net /amp.~fault~ renamed /amp.~{fault}
- net /amp.~gain0~ renamed /amp.~{gain0}
- net /amp.~gain1~ renamed /amp.~{gain1}
- net /dac.~connected~ renamed /dac.~{connected}
- net /main.~jackconn~ renamed /main.~{jackconn}
- net /~icsp.res~ renamed /~{icsp.res}
- net /~mcu.res~ renamed /~{mcu.res}
Other:
- net class Default removed
